File: Watch/rgbwatch/_autosave-rgbwatch.sch (KiCad schematic (older format))
At the start: 72 parts, among them J1 USB_B_Micro, J2 NRST, J3 SWCLK, J4 SWDIO, J5 UART2_TX, J6 UART2_RX, Q1 p-channel, Q2 n-channel, Q3 n-channel, U1 LP5024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

Commit message: Add files via upload
Parts:
- added R19, R20: 10K, Resistor_SMD:R_0603_1608Metric, symbol Device:R_Small
Connections:
- net GND: now also R19.2, R20.2
- net S1: now also Q2.1 (G), R19.1
- net S2: now also Q3.1 (G), R20.1
Changed lines of the file:
@@
 U 1 1 5FFA87A0
 P 1250 3250
-F 0 "Q2" V 1399 3150 50  0000 C CNN
-F 1 "n-channel" V 1490 3150 50  0000 C CNN
+F 0 "Q2" V 1300 3000 50  0000 C CNN
+F 1 "n-channel" V 1400 3200 50  0000 C CNN
 F 2 "Package_TO_SOT_SMD:SOT-23" H 1250 3650 50  0001 C CNN
 F 3 "" H 1250 3650 50  0001 C CNN
@@
 U 1 1 5FD0CDFB
 P 1300 3850
-F 0 "Q3" V 1449 3750 50  0000 C CNN
-F 1 "n-channel" V 1540 3750 50  0000 C CNN
+F 0 "Q3" V 1400 3600 50  0000 C CNN
+F 1 "n-channel" V 1450 3800 50  0000 C CNN
 F 2 "Package_TO_SOT_SMD:SOT-23" H 1300 4250 50  0001 C CNN
 F 3 "" H 1300 4250 50  0001 C CNN
@@
 	0    1    1    0
 $EndComp
+$Comp
+L Device:R_Small R19
+U 1 1 5FD68C88
+P 1250 2950
+F 0 "R19" V 1200 2700 50  0000 C CNN
+F 1 "10K" V 1300 2700 50  0000 C CNN
+F 2 "Resistor_SMD:R_0603_1608Metric" H 1250 2950 50  0001 C CNN
+F 3 "~" H 1250 2950 50  0001 C CNN
+	1    1250 2950
+	0    -1   -1   0
+$EndComp
+$Comp
+L Device:R_Small R20
+U 1 1 5FD69596
+P 1300 3550
+F 0 "R20" V 1250 3300 50  0000 C CNN
+F 1 "10K" V 1350 3300 50  0000 C CNN
+F 2 "Resistor_SMD:R_0603_1608Metric" H 1300 3550 50  0001 C CNN
+F 3 "~" H 1300 3550 50  0001 C CNN
+	1    1300 3550
+	0    -1   -1   0
+$EndComp
+$Comp
+L power:GND #PWR06
+U 1 1 5FD69C0C
+P 1350 2950
+F 0 "#PWR06" H 1350 2700 50  0001 C CNN
+F 1 "GND" H 1355 2777 50  0000 C CNN
+F 2 "" H 1350 2950 50  0001 C CNN
+F 3 "" H 1350 2950 50  0001 C CNN
+	1    1350 2950
+	1    0    0    -1
+$EndComp
+$Comp
+L power:GND #PWR07
+U 1 1 5FD6A3D7
+P 1400 3550
+F 0 "#PWR07" H 1400 3300 50  0001 C CNN
+F 1 "GND" H 1405 3377 50  0000 C CNN
+F 2 "" H 1400 3550 50  0001 C CNN
+F 3 "" H 1400 3550 50  0001 C CNN
+	1    1400 3550
+	1    0    0    -1
+$EndComp
+Text GLabel 1150 2950 0    50   Input ~ 0
+S1
+Text GLabel 1200 3550 0    50   Input ~ 0
+S2
 $EndSCHEMATC
