File: Watch/rgbwatch/rgbwatch.kicad_pcb (KiCad board)
At the start: 4 copper layers, 40 x 40 mm, 74 parts, among them J2 NRST, J3 SWCLK, J4 SWDIO, J5 UART2_TX, J6 UART2_RX, Q1 p-channel, Q2 2N7000, Q2 n-channel, Q3 n-channel, U1 LP5024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

Commit message: Add files via upload
Parts:
- added J1: USB_B_Micro, Connector_USB:USB_Micro-B_Amphenol_10104110_Horizontal, B.Cu at (160.1, 75.0)
- added J10: I2C2_SCL, Connector_Wire:SolderWirePad_1x01_SMD_1x2mm, B.Cu at (173.8, 91.3)
- added J11: I2C1_SDA, Connector_Wire:SolderWirePad_1x01_SMD_1x2mm, B.Cu at (176.2, 91.3)
- added J12: I2C1_SCL, Connector_Wire:SolderWirePad_1x01_SMD_1x2mm, B.Cu at (178.5, 91.3)
- added J7: +BATT, Connector_Wire:SolderWirePad_1x01_SMD_1x2mm, B.Cu at (171.4, 58.4)
- added J8: -BATT, Connector_Wire:SolderWirePad_1x01_SMD_1x2mm, B.Cu at (177.8, 58.4)
- added J9: I2C2_SDA, Connector_Wire:SolderWirePad_1x01_SMD_1x2mm, B.Cu at (171.4, 91.3)
- J2, J3, J4, J5, J6: footprint rgbwatch:headerpin -> Connector_Wire:SolderWirePad_1x01_SMD_1x2mm; moved to B.Cu
- Q2, U3: moved to F.Cu
- R1: value 0R -> 10K
- moved R13 125.5 mm to (184.0, 67.5)
- moved J5 109.2 mm to (191.6, 72.2), turned to 270 degrees
- moved J6 109.1 mm to (191.6, 69.9), turned to 270 degrees
- moved Y1 105.4 mm to (175.0, 79.0)
- moved J2 102.4 mm to (191.6, 79.3), turned to 270 degrees
- moved J4 101.2 mm to (191.6, 74.6), turned to 270 degrees
- moved J3 97.1 mm to (191.6, 77.0), turned to 270 degrees
- moved Q3 89.0 mm to (187.8, 82.8)
- moved U3 88.5 mm to (170.0, 72.0)
- moved Q2 87.9 mm to (170.8, 59.9), turned to 90 degrees
- moved U4 80.6 mm to (176.4, 74.9), turned to 90 degrees
- moved Q1 76.4 mm to (164.4, 71.8), turned to 180 degrees
- moved U6 75.2 mm to (175.0, 69.5)
- moved R3 61.6 mm to (165.8, 65.5)
- moved D1 58.9 mm to (164.6, 77.0), turned to 90 degrees
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Connections:
- C2 pad 1: Net-(C2-Pad1) -> VCC
- L1 pad 2: Net-(C2-Pad1) -> VCC
- R1 pad 1: Net-(C2-Pad1) -> SWDIO
- R1 pad 2: VCC -> GND
- U2 pad 5: Net-(C2-Pad1) -> VCC
- U4 pad 25: Net-(U4-Pad25) -> CTRL
Routing:
- net Net-(C1-Pad1): track 0.00 -> 10.3 mm, vias 0 -> 4
- net Net-(L1-Pad1): track 0.00 -> 2.97 mm
- net CTRL: track 0.00 -> 0.85 mm, vias 0 -> 1
- net VCC: vias 0 -> 3
- net GND: vias 0 -> 2
- added copper zone on F.Cu, net GND
- added copper zone on In1.Cu, net GND
- added copper zone on F.Cu, net Net-(C1-Pad1)
- added copper zone on F.Cu, net VBUS
- added copper zone on F.Cu, net VCC
Other:
- net class Default: via_dia 0.8 -> 0.5; via_drill 0.4 -> 0.3

Commit message: Add files via upload
Parts:
- removed the Q2 at (170.8, 59.9)
- removed the Q2 at (140.0, 82.0)
- added Q2: n-channel, Package_TO_SOT_SMD:SOT-23, F.Cu at (168.2, 75.9)
- added R21: 10K, Resistor_SMD:R_0402_1005Metric, F.Cu at (179.6, 82.6)
- A0, A1, A2, A3, A4, A5, A6, A7, B0, B1, B2, B3, L1, U1, U2, U3, U5, U6: moved to B.Cu
- C1, C10, C11, C12, C14, C15, C16, C2, C5: footprint Capacitor_SMD:C_0603_1608Metric -> Capacitor_SMD:C_0402_1005Metric; moved to B.Cu
- C13, C3, C4, C6, C7, C8, C9: footprint Capacitor_SMD:C_0603_1608Metric -> Capacitor_SMD:C_0402_1005Metric
- J1, J10, J11, J12, J2, J3, J4, J5, J6, J7, J8, J9: moved to F.Cu
- R1, R10, R11, R12, R13, R14, R15, R16, R17, R18, R4, R7, R8, R9, Rprog1: footprint Resistor_SMD:R_0603_1608Metric -> Resistor_SMD:R_0402_1005Metric
- R19, R2, R20, R3, R5, R6: footprint Resistor_SMD:R_0603_1608Metric -> Resistor_SMD:R_0402_1005Metric; moved to B.Cu
- moved B7 121.0 mm to (167.2, 34.1)
- moved C15 117.0 mm to (178.2, 73.5), turned to 90 degrees
- moved B4 114.4 mm to (154.6, 32.8)
- moved B5 113.2 mm to (156.8, 29.0)
- moved B6 105.8 mm to (163.1, 33.8)
- moved A6 101.8 mm to (169.8, 60.2)
- moved A3 95.5 mm to (188.6, 73.1)
- moved A0 94.7 mm to (174.8, 60.2)
- moved B2 93.7 mm to (159.4, 65.8)
- moved A2 92.0 mm to (187.9, 66.5)
- moved C14 88.5 mm to (178.7, 77.2), turned to 180 degrees
- moved A4 87.9 mm to (188.2, 79.2)
- moved B3 74.7 mm to (164.2, 61.4)
- moved BATI1 74.2 mm to (181.4, 87.5)
- moved A5 70.2 mm to (185.0, 87.0)
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Connections:
- R11 pad 1: GND -> VCC
- R5 pad 2: +BATT -> VCC
- R6 pad 1: +BATT -> VCC
- R6 pad 2: I2C2_SCL -> I2C1_SCL
- R7 pad 2: GND -> VCC
- U3 pad 4: ALARMB -> -BATT
- U3 pad 8: I2C2_SCL -> I2C1_SCL
- U4 pad 22: VSEL1 -> VSEL3
- U4 pad 24: VSEL3 -> VSEL1
- U4 pad 26: I2C2_SCL -> I2C1_SCL
- U4 pad 28: Net-(U4-Pad28) -> ALARMB
Routing:
- net CTRL: track 0.85 -> 25.7 mm, vias 1 -> 3
- net VSEL1: track 0.00 -> 16.6 mm, vias 0 -> 1
- net VSEL3: track 0.00 -> 15.9 mm, vias 0 -> 1
- net VSEL2: track 0.00 -> 15.8 mm, vias 0 -> 1
- net VCC: track 0.00 -> 12.5 mm, vias 3 -> 1
- net I2C2_SDA: track 0.00 -> 10.6 mm, vias 0 -> 2
- net I2C1_SCL: track 0.00 -> 10.3 mm, vias 0 -> 1
- net GND: track 0.00 -> 10.1 mm, vias 2 -> 9
- net Net-(C1-Pad1): track 10.3 -> 1.23 mm, vias 4 -> 0
- net I2C1_SDA: track 0.00 -> 7.75 mm, vias 0 -> 1
- net -BATT: track 0.00 -> 6.66 mm
- net I2C2_SCL: track 0.00 -> 6.66 mm, vias 0 -> 2
- net Vled: track 0.00 -> 4.85 mm, vias 0 -> 1
- net +BATT: track 0.00 -> 4.06 mm
- net OSC32_IN: track 0.00 -> 3.52 mm
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- removed copper zone on F.Cu, net Net-(C1-Pad1)
- removed copper zone on F.Cu, net VBUS
- removed copper zone on F.Cu, net VCC
Other:
- rule trace_min: 0.2 -> 0.15
