File: Watch/rgbwatch/rgbwatch.sch (KiCad schematic (older format))
At the start: 29 parts, among them Q1 2N7002H

Commit message: Add files via upload
Parts:
- removed Ch: UHD1110-FKA, symbol rgbwatch:UHD1110-FKA
- removed D?: D_Schottky, symbol Device:D_Schottky
- removed Q1: 2N7002H, Package_TO_SOT_SMD:SOT-23, symbol Transistor_FET:2N7002H
- removed U?: LIS2DH12TR, digikey-footprints:VFLGA-12_2x2mm, symbol dk_Motion-Sensors-Accelerometers:LIS2DH12TR
- removed U?: LP5024, symbol rgbwatch:LP5024
- added C? (x2): 10uF, symbol Device:C_Small
- added C? (x3): 100nF, symbol Device:C_Small
- added C? (x2): 4.7uF, symbol Device:C_Small
- added Ch0 (x8), Ch1 (x8), Ch?: UHD1110-FKA, symbol rgbwatch:UHD1110-FKA
- added D?: D_Schottky, symbol Device:D_Schottky
- added FB?: Ferrite_Bead, symbol Device:Ferrite_Bead
- added Q?: TP0610T, Package_TO_SOT_SMD:SOT-23, symbol Transistor_FET:TP0610T
- added Q? (x2): 2N7000, Package_TO_SOT_THT:TO-92_Inline, symbol Transistor_FET:2N7000
- added R? (x3): 10K, symbol Device:R_Small
- added R? (x2): 4.7K, symbol Device:R_Small
- added SW?: SW_Push, symbol Switch:SW_Push
- added U?: LIS3DH, Package_LGA:LGA-16_3x3mm_P0.5mm_LayoutBorder3x5y, symbol Sensor_Motion:LIS3DH
- added Y?: 32.768 KHz, symbol Device:Crystal_Small
Connections:
- net labels added: B0, B1, B2, B3, B4, B5, B6, B7, CH0, CH1, G0, G1, G2, G3, G4, G5, G6, G7, I2C1_SDA, I2C2_SCL, I2C2_SDA, INT1, INT2, NRST, OSC32_IN, OSC32_OUT, R0, R1, R2, R3, R4, R5, R6, R7, S1, S2, SWCLK, SWDIO, UART2_RX, UART2_TX
- net labels removed: SCL1, SDA1
- wire segments 51 -> 108
Other:
- note added: "CHANGE PINS OF MOSFET\n"
- note added: "Connect SW to MCU and Load to Vled which can be turned on and off power saving mode lol\n"
- moved on the sheet: C?, J?, R?, TH1, U?

Commit message: Add files via upload
Parts:
- removed C?: C_Small, symbol Device:C_Small
- removed L?: L_Small, symbol Device:L_Small
- removed Q? (x2): 2N7000, Package_TO_SOT_THT:TO-92_Inline, symbol Transistor_FET:2N7000
- removed R?: R_Small, symbol Device:R_Small
- removed SW?: SW_Push, symbol Switch:SW_Push
- removed U?: USBLC6-2SC6, Package_TO_SOT_SMD:SOT-23-6, symbol Power_Protection:USBLC6-2SC6
- added C13, C14, C15, C16: 10uF, Capacitor_SMD:C_0603_1608Metric, symbol Device:C_Small
- added J2: NRST, rgbwatch:headerpin, symbol Connector:Conn_01x01_Male
- added J3: SWCLK, rgbwatch:headerpin, symbol Connector:Conn_01x01_Male
- added J4: SWDIO, rgbwatch:headerpin, symbol Connector:Conn_01x01_Male
- added J5: UART2_TX, rgbwatch:headerpin, symbol Connector:Conn_01x01_Male
- added J6: UART2_RX, rgbwatch:headerpin, symbol Connector:Conn_01x01_Male
- added Q2, Q3: n-channel, Package_TO_SOT_SMD:SOT-23, symbol rgbwatch:n-channel
- added R12, R17, R? (x2): 10K, Resistor_SMD:R_0603_1608Metric, symbol Device:R_Small
- added R13: 0R, Resistor_SMD:R_0603_1608Metric, symbol Device:R_Small
- added R14, R16: 4.7K, Resistor_SMD:R_0603_1608Metric, symbol Device:R_Small
- added R15: IREF, Resistor_SMD:R_0603_1608Metric, symbol Device:R_Small
- added R18: IN_EN, Resistor_SMD:R_0603_1608Metric, symbol Device:R_Small
- A0, A1, A2, A3, A4, A5, A6, A7: renamed from Ch0; footprint (none) -> rgbwatch:UHD1110-FKA
- B0, B1, B2, B3, B4, B5, B6, B7: renamed from Ch1; footprint (none) -> rgbwatch:UHD1110-FKA
- BATI1: renamed from Ch?; footprint (none) -> rgbwatch:UHD1110-FKA
- C1, C2: footprint (none) -> Capacitor_SMD:C_0603_1608Metric
- C10, C11, C12, C3, C4, C5, C6, C7, C8, C9: renamed from C?; footprint (none) -> Capacitor_SMD:C_0603_1608Metric
- D1: renamed from D?; footprint (none) -> Diode_SMD:D_SOD-123
- FB1: renamed from FB?; footprint (none) -> Inductor_SMD:L_0603_1608Metric
- L1: renamed from L?; footprint (none) -> Inductor_SMD:L_0805_2012Metric
- Q1: renamed from Q?; value TP0610T -> p-channel
- R1, R2, R3, TH1: footprint (none) -> Resistor_SMD:R_0603_1608Metric
- R10, R11, R4, R5, R6, R7, R8, R9: renamed from R?; footprint (none) -> Resistor_SMD:R_0603_1608Metric
- Rprog1: renamed from Rprog; footprint (none) -> Resistor_SMD:R_0603_1608Metric
- U1: renamed from U?; footprint (none) -> rgbwatch:QFN-32_EP_4.4x4.4_Pitch0.4mm
- U2: renamed from U?; footprint (none) -> Package_SON:WSON-12-1EP_3x2mm_P0.5mm_EP1x2.65_ThermalVias
- U3: renamed from U?; footprint (none) -> rgbwatch:WDFN-8
- U4: renamed from U?; footprint (none) -> rgbwatch:QFN-28_EP_5.3x5.3_Pitch0.5mm
- U5: renamed from U?; footprint (none) -> Package_DFN_QFN:DFN-10-1EP_3x3mm_P0.5mm_EP1.65x2.38mm_ThermalVias
- Y1: renamed from Y?; footprint (none) -> Crystal:Crystal_SMD_2012-2Pin_2.0x1.2mm
- gave numbers to parts that had none: 2
Connections:
- net CH0: now also Q2.2 (S)
- net CH1: now also Q3.2 (S)
- net GND: now also C11.1, J1.5 (GND), U1.25 (ADDR0), U1.26 (ADDR1), U1.33 (GND), C13.2, C14.1, C15.2, C16.1, R12.2, R13.2, R15.1, R17.2, R?.2, R?.2; no longer C11.2, U6.7 (SDO/SA0)
- net I2C2_SCL: now also U1.29 (SCL), R16.2
- net I2C2_SDA: now also U1.28 (SDA), R14.2
- net NRST: now also J2.1 (Pin_1), R13.1
- net S1: now also Q2.1 (G), R?.1
- net S2: now also Q3.1 (G), R?.1
- net SWCLK: now also J3.1 (Pin_1), R12.1
- net SWDIO: now also J4.1 (Pin_1)
- net UART2_RX: now also J6.1 (Pin_1)
- net UART2_TX: now also J5.1 (Pin_1)
- net VBUS: now also C13.1
- net VCC: now also C11.2, U1.27 (VCC), C15.1, C16.2, R14.1, R16.1, R18.2; no longer C11.1
- net VSEL1: now also U4.22 (PD0)
- net VSEL2: now also U4.23 (PD1)
- net VSEL3: now also U4.24 (PD2)
- net Vled: now also Q2.3 (D), Q3.3 (D)
- net IN_EN: now reaches U1.30 (IN_EN)
- net IN_EN: now also R18.1
- net at U1.31 (IREF): now also R15.2
- net at U1.32 (VCAP): now also C14.2
- new net: R17.1, U6.7 (SDO/SA0)
- no-connect marks 0 -> 17
Other:
- note added: "LIS3DH"
- note added: "Linear LiPo Charger"
- moved on the sheet: A0, A1, A2, A3, A4, A5, A6, A7, B0, B1, B2, B3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

Commit message: Add files via upload
Parts:
- gave numbers to parts that had none: 2
Changed lines of the file:
@@
 $EndComp
 $Comp
-L Device:R_Small R?
+L Device:R_Small R19
 U 1 1 5FD68C88
 P 1250 2950
-F 0 "R?" V 1200 2700 50  0000 C CNN
+F 0 "R19" V 1200 2700 50  0000 C CNN
 F 1 "10K" V 1300 2700 50  0000 C CNN
 F 2 "Resistor_SMD:R_0603_1608Metric" H 1250 2950 50  0001 C CNN
@@
 $EndComp
 $Comp
-L Device:R_Small R?
+L Device:R_Small R20
 U 1 1 5FD69596
 P 1300 3550
-F 0 "R?" V 1250 3300 50  0000 C CNN
+F 0 "R20" V 1250 3300 50  0000 C CNN
 F 1 "10K" V 1350 3300 50  0000 C CNN
 F 2 "Resistor_SMD:R_0603_1608Metric" H 1300 3550 50  0001 C CNN
@@
 $EndComp
 $Comp
-L power:GND #PWR?
+L power:GND #PWR06
 U 1 1 5FD69C0C
 P 1350 2950
-F 0 "#PWR?" H 1350 2700 50  0001 C CNN
+F 0 "#PWR06" H 1350 2700 50  0001 C CNN
 F 1 "GND" H 1355 2777 50  0000 C CNN
 F 2 "" H 1350 2950 50  0001 C CNN
@@
 $EndComp
 $Comp
-L power:GND #PWR?
+L power:GND #PWR07
 U 1 1 5FD6A3D7
 P 1400 3550
-F 0 "#PWR?" H 1400 3300 50  0001 C CNN
+F 0 "#PWR07" H 1400 3300 50  0001 C CNN
 F 1 "GND" H 1405 3377 50  0000 C CNN
 F 2 "" H 1400 3550 50  0001 C CNN

Commit message: Add files via upload
Parts:
- added J10: I2C2_SCL, Connector_Wire:SolderWirePad_1x01_SMD_1x2mm, symbol Connector:Conn_01x01_Male
- added J11: I2C1_SDA, Connector_Wire:SolderWirePad_1x01_SMD_1x2mm, symbol Connector:Conn_01x01_Male
- added J12: I2C1_SCL, Connector_Wire:SolderWirePad_1x01_SMD_1x2mm, symbol Connector:Conn_01x01_Male
- added J7: +BATT, Connector_Wire:SolderWirePad_1x01_SMD_1x2mm, symbol Connector:Conn_01x01_Male
- added J8: -BATT, Connector_Wire:SolderWirePad_1x01_SMD_1x2mm, symbol Connector:Conn_01x01_Male
- added J9: I2C2_SDA, Connector_Wire:SolderWirePad_1x01_SMD_1x2mm, symbol Connector:Conn_01x01_Male
- J1: footprint (none) -> Connector_USB:USB_Micro-B_Amphenol_10104110_Horizontal; symbol Connector:USB_B_Micro -> rgbwatch-rescue:USB_B_Micro-Connector
- J2, J3, J4, J5, J6: footprint rgbwatch:headerpin -> Connector_Wire:SolderWirePad_1x01_SMD_1x2mm
- R1: value 0R -> 10K
Connections:
- net +BATT: now also J7.1 (Pin_1)
- net -BATT: now also J8.1 (Pin_1)
- net ALARMB: now also U4.28 (PB8)
- net CTRL: now also U4.25 (PD3)
- net GND: now also R1.2
- net I2C1_SDA: now also J11.1 (Pin_1)
- net I2C2_SCL: now also J10.1 (Pin_1)
- net I2C2_SDA: now also J9.1 (Pin_1)
- net SWDIO: now also R1.1
- net VCC: now also C2.1, L1.2, U2.5 (VOUT); no longer R1.2
- new net I2C1_SCL: J12.1 (Pin_1)
- no-connect marks 17 -> 15
Other:
- moved on the sheet: C13, FB1, J1, J2, J3, J4, J5, J6, R12, TH1

Commit message: Add files via upload
Parts:
- added R21: 10K, Resistor_SMD:R_0402_1005Metric, symbol Device:R_Small
- C1, C10, C11, C12, C13, C14, C15, C16, C2, C3, C4, C5, C6, C7, C8, C9: footprint Capacitor_SMD:C_0603_1608Metric -> Capacitor_SMD:C_0402_1005Metric
- R1, R10, R11, R12, R13, R14, R15, R16, R17, R18, R19, R2, R20, R3, R4, R5, R6, R7, R8, R9, Rprog1: footprint Resistor_SMD:R_0603_1608Metric -> Resistor_SMD:R_0402_1005Metric
Connections:
- net +BATT: no longer R5.2, R6.1
- net -BATT: now also U3.4 (ALARMB)
- net ALARMB: no longer U3.4 (ALARMB)
- net CTRL: now also R21.2
- net GND: now also R21.1; no longer R11.1, R7.2
- net I2C1_SCL: now also R6.2, U3.8 (SCL), U4.26 (PB6)
- net I2C2_SCL: no longer R6.2, U3.8 (SCL), U4.26 (PB6)
- net VCC: now also R11.1, R5.2, R6.1, R7.2
- net VSEL1: now also U4.24 (PD2); no longer U4.22 (PD0)
- net VSEL3: now also U4.22 (PD0); no longer U4.24 (PD2)
