File: Watch/rgbwatch/rgbwatch_1.kicad_pcb (KiCad board)
At the start: 4 copper layers, 40 x 40 mm, 81 parts, among them J1 USB_B_Micro, J10 I2C2_SCL, J11 I2C1_SDA, J12 I2C1_SCL, J2 NRST, J3 SWCLK, J4 SWDIO, J5 UART2_TX, J6 UART2_RX, J7 +BATT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

Commit message: Add files via upload
Parts:
- moved C6 56.4 mm to (239.6, 111.6)
- moved R13 35.0 mm to (213.4, 103.1), turned to 0 degrees
- moved C2 0.25 mm to (166.3, 77.9)
- moved R6 0.25 mm to (179.6, 81.3)
- moved C8 0.10 mm to (186.4, 79.4)
- moved R5 0.10 mm to (179.6, 80.4)
- moved R3 0.08 mm to (179.6, 78.4)
- moved C14 0.05 mm to (178.7, 77.2)
Routing:
- net -BATT: track 6.66 -> 0.00 mm
- net VCC: track 8.91 -> 2.43 mm
- net GND: track 4.81 -> 1.51 mm, vias 3 -> 1
- net OSC32_OUT: track 2.13 -> 0.00 mm
- net OSC32_IN: track 1.99 -> 0.00 mm
- net CTRL: track 24.1 -> 22.2 mm, vias 3 -> 2
- net G1: track 1.62 -> 0.00 mm, vias 1 -> 0
- net Net-(C14-Pad2): track 1.60 -> 0.00 mm
- net B1: track 1.55 -> 0.00 mm, vias 1 -> 0
- net +BATT: track 1.47 -> 0.00 mm
- net R0: track 1.45 -> 0.00 mm, vias 1 -> 0
- net Net-(C1-Pad1): track 1.23 -> 2.63 mm
- net R1: track 1.36 -> 0.00 mm, vias 1 -> 0
- net B2: track 1.27 -> 0.00 mm, vias 1 -> 0
- net VSEL1: track 16.6 -> 15.3 mm
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Other:
- rule trace_min: 0.15 -> 0.2
